File: noise-collector/_autosave-savox noise collector.kicad_pcb (KiCad board)
At the start: 4 copper layers, 39.4 x 50.5 mm, 65 parts, among them J1 Conn_01x02_Pin, J2 USB_C_Receptacle_USB2.0_16P, Q4 2N7002NXAKR, U1 ESP32-S3, U2 TPS7A0333PDQNR3, U3 OPA1679IDR, U6 TPS2113ADRBR, Y2 CC7V-T1A-32.768KHZ-9PF-20PPM-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, Y3 Crystal_GND24

Commit message: Add files via upload
Parts:
- removed D3: 1N4148W, Diode_SMD:D_SOD-123
- removed MIC1: IMP23ABSUTR, SamacSys_Parts:RHLGA5_3P5X2P65X0P98_STM
- added D5: NSR0320MW2T1G, SamacSys_Parts:SOD2512X110N, F.Cu at (170.4, 85.7)
- added U4: TP6004-TR, SamacSys_Parts:TSSOP-14_TPK-L, F.Cu at (147.5, 112.8)
- J1: footprint Connector_PinHeader_1.27mm:PinHeader_1x02_P1.27mm_Horizontal -> Connector_PinHeader_2.54mm:PinHeader_1x02_P2.54mm_Horizontal
- R14: value 3313J-1-204E -> 220k; footprint SamacSys_Parts:TRIM_3313J-1-204E -> Resistor_SMD:R_0402_1005Metric
- R2: value 150k -> 220k; footprint Resistor_SMD:R_0201_0603Metric -> Resistor_SMD:R_0402_1005Metric
- U2: value TPS7A0333PDQNR3 -> C5220177
- U3: value OPA1679IDR -> ~; footprint SamacSys_Parts:SOIC127P600X175-14N -> OwnFootprints:OwnMIcrophone
- moved U3 23.2 mm to (166.7, 99.6), turned to 180 degrees
- moved C7 11.1 mm to (160.9, 94.9), turned to 90 degrees
- moved R12 5.57 mm to (153.9, 116.8), turned to 0 degrees
- moved C10 4.77 mm to (165.3, 103.3)
- moved R14 3.62 mm to (155.6, 116.9), turned to 0 degrees
- moved ANT2 3.05 mm to (162.8, 117.7), turned to -90 degrees
- moved D8 2.56 mm to (151.2, 116.8)
- moved L3 2.52 mm to (156.4, 110.9), turned to 90 degrees
- moved D4 2.02 mm to (140.9, 111.7)
- moved D2 2.00 mm to (138.6, 111.7)
- moved R7 1.92 mm to (142.7, 111.2)
- moved R10 1.92 mm to (143.5, 111.2)
- moved R2 1.89 mm to (151.6, 111.1), turned to 90 degrees
- moved R11 1.85 mm to (142.8, 113.8)
- moved R5 1.83 mm to (143.5, 114.5)
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Connections:
- R10 pad 2: Net-(U3--INA) -> Net-(U4-INA-)
- R11 pad 2: Net-(U3--INB) -> Net-(U4-INB-)
- R12 pad 2: /D_OP+ -> Net-(U4-IND+)
- R13 pad 1: Net-(U3--INC) -> Net-(U4-INC-)
- R13 pad 2: Net-(U3--IND) -> Net-(U4-IND-)
- R14 pad 1: /D_OP+ -> Net-(U4-IND+)
- R2 pad 1: /Amp_out -> Net-(U4-IND-)
- R2 pad 2: Net-(U3--IND) -> /Amp_out
- R5 pad 2: Net-(U3--INB) -> Net-(U4-INB-)
- R7 pad 2: Net-(U3--INA) -> Net-(U4-INA-)
- U3 pad 1: Net-(D7-A) -> /MCO
- U3 pad 2: Net-(U3--INA) -> GND
- U3 pad 3: Net-(D2-A) -> GND
Routing:
- net Net-(U6-IN1): track 12.7 -> 42.4 mm, vias 0 -> 2
- net Net-(U4-IND+): track 0.00 -> 12.6 mm
- net Net-(U3--IND): track 12.4 -> 0.00 mm
- net /3V3: track 108.3 -> 120.4 mm, vias 5 -> 7
- net /D_OP+: track 12.0 -> 0.00 mm
- net GND: track 54.1 -> 43.2 mm, vias 9 -> 331
- net Net-(U4-IND-): track 0.00 -> 5.69 mm
- net Net-(D7-K): track 8.28 -> 3.43 mm
- net Net-(ANT2-FEED): track 8.39 -> 4.24 mm
- net Net-(U1-XTAL_N): track 14.4 -> 10.7 mm
- net Net-(U3--INB): track 3.02 -> 0.00 mm
- net Net-(U3--INC): track 3.02 -> 0.00 mm
- net Net-(U3--INA): track 2.60 -> 0.00 mm
- net Net-(D7-A): track 20.8 -> 18.4 mm, vias 2 -> 3
- net Net-(D8-A): track 9.48 -> 7.31 mm
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Other:
- board text added: "Savox noise collector PCB Designed by Ilkka Etula and Nhat Hong Protopaja 2024"
- board text removed: "Savox noise collector PCB Designed by Ilkka Etula and Nhat Hong"
