File: noise-collector/_autosave-savox noise collector.kicad_sch (KiCad schematic)
At the start: 65 parts, among them J1 Conn_01x02_Pin, J2 USB_C_Receptacle_USB2.0_16P, Q4 2N7002NXAKR, U1 ESP32-S3, U2 TPS7A0333PDQNR3, U3 OPA1679IDR, U6 TPS2113ADRBR, Y2 CC7V-T1A-32.768KHZ-9PF-20PPM-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, Y3 Crystal_GND24

Commit message: Add files via upload
Parts:
- removed D3: 1N4148W, Diode_SMD:D_SOD-123, symbol Diode:1N4148W
- removed MIC1: IMP23ABSUTR, SamacSys_Parts:RHLGA5_3P5X2P65X0P98_STM, symbol 2024-07-29_12-07-10:IMP23ABSUTR
- removed R14: 3313J-1-204E, SamacSys_Parts:TRIM_3313J-1-204E, symbol 3313J-1-204E:3313J-1-204E
- removed U3: OPA1679IDR, SamacSys_Parts:SOIC127P600X175-14N, symbol OPA1679IDR:OPA1679IDR
- added D5: NSR0320MW2T1G, SamacSys_Parts:SOD2512X110N, symbol NSR0320MW2T1G:NSR0320MW2T1G
- added R14: 220k, Resistor_SMD:R_0402_1005Metric, symbol Device:R
- added U3: ~, OwnFootprints:OwnMIcrophone, symbol ProLibrary_pcs_2024-07-25:LMA2718T421-OA5-2
- added U4: TP6004-TR, SamacSys_Parts:TSSOP-14_TPK-L, symbol 2024-08-12_07-45-24:TP6004-TR
- ANT2: LCSC Part (none) -> C127629
- BT1: LCSC Part (none) -> C964831
- Boot1, Reset1: LCSC Part (none) -> C2888954
- C1, C11, C17, C23, C24, C3, C6, C7: LCSC Part (none) -> C1525
- C10, C13, C19, C20, C21, C22, C25: LCSC Part (none) -> C315248
- C12, C18, C2, C27, C4, C5, C8, C9: LCSC Part (none) -> C52923
- C14: LCSC Part (none) -> C1551
- C15, C16: LCSC Part (none) -> C1578
- C26: LCSC Part (none) -> C76903
- D1: LCSC Part (none) -> C3646921
- D2, D4, D7, D8: LCSC Part (none) -> C48192
- J1: footprint Connector_PinHeader_1.27mm:PinHeader_1x02_P1.27mm_Horizontal -> Connector_PinHeader_2.54mm:PinHeader_1x02_P2.54mm_Horizontal; now not fitted
- J2: LCSC Part (none) -> C319148
- L1: LCSC Part (none) -> C18216
- L2: LCSC Part (none) -> C275281
- L3: LCSC Part (none) -> C74301
- Q4: LCSC Part (none) -> C551416
- R1, R9: LCSC Part (none) -> C25519
- R10, R11, R12, R13, R15, R4, R5, R7: LCSC Part (none) -> C102685
- R2: value 150k -> 220k; footprint Resistor_SMD:R_0201_0603Metric -> Resistor_SMD:R_0402_1005Metric; LCSC Part (none) -> C25767
- R3: LCSC Part (none) -> C473048
- R6, R8: LCSC Part (none) -> C274341
- U1: LCSC Part (none) -> C2913196
- U2: value TPS7A0333PDQNR3 -> C5220177; LCSC Part (none) -> C5220177
- U6: LCSC Part (none) -> C354512
- Y2: LCSC Part (none) -> C337577
- Y3: LCSC Part (none) -> C387435
Connections:
- net 3V3: now also D5.1 (K), U3.4 (VDD), U4.4 (VS+)
- net Amp_out: now also R2.2, U4.14 (OUTD); no longer R2.1
- net GND: now also R14.2, U3.2 (GND), U3.3 (GND), U4.11 (VS-)
- net MCO: now also U3.1 (OUT)
- net at D2.1 (K), R15.2: now also U4.10 (INC+)
- net at D8.2 (A), R5.1: now also U4.7 (OUTB)
- net at R11.2, R5.2: now also U4.6 (INB-)
- net at R10.2, R7.2: now also U4.2 (INA-)
- net at R13.1: now also U4.8 (OUTC), U4.9 (INC-)
- net at R13.2: now also R2.1, U4.13 (IND-); no longer R2.2
- net at J1.1 (Pin_1), Q4.3 (D): now also D5.2 (A)
- net at D7.2 (A), R10.1, R11.1: now also U4.1 (OUTA)
- net at D2.2 (A), D4.1 (K): now also U4.3 (INA+), U4.5 (INB+)
- net D_OP+: no longer names the net of R12.2
- net D_OP+: now also R14.1, U4.12 (IND+)
Other:
- moved on the sheet: R13, R2
